Commit message: added ROS description and moveit config packages

File: src/robotic_arm_description/urdf/robotic_arm.xacro (robot description, xacro)
@@ -5,9 +5,4 @@
 <xacro:include filename="$(find robotic_arm_description)/urdf/robotic_arm.gazebo" />
 <link name="base_link">
-  <inertial>
-    <origin rpy="0 0 0" xyz="-7.044926902746826e-09 -4.737750495934672e-09 0.038474409050025755"/>
-    <mass value="5.749401825671835"/>
-    <inertia ixx="0.007412" ixy="-0.0" ixz="-0.0" iyy="0.007412" iyz="-0.0" izz="0.008288"/>
-  </inertial>
   <visual>
     <origin rpy="0 0 0" xyz="0 0 0"/>
@@ -26,10 +21,10 @@
 <link name="link1_1">
   <inertial>
-    <origin rpy="0 0 0" xyz="-0.014019658312986 0.001532580028955315 0.09630243018941843"/>
+    <origin rpy="0 0 0" xyz="-0.014103177682961474 2.911659828472621e-08 0.09630243018941843"/>
     <mass value="9.886638889856904"/>
-    <inertia ixx="0.028946" ixy="7.7e-05" ixz="0.002237" iyy="0.029643" iyz="-0.000245" izz="0.010294"/>
-  </inertial>
-  <visual>
-    <origin rpy="0 0 0" xyz="0.0 0.0 -0.082"/>
+    <inertia ixx="0.028938" ixy="0.0" ixz="0.00225" iyy="0.029652" iyz="0.0" izz="0.010294"/>
+  </inertial>
+  <visual>
+    <origin rpy="0 0 0" xyz="-0.0 -0.0 -0.082"/>
     <geometry>
       <mesh filename="package://robotic_arm_description/meshes/link1_1.stl" scale="0.001 0.001 0.001"/>
@@ -38,5 +33,5 @@
   </visual>
   <collision>
-    <origin rpy="0 0 0" xyz="0.0 0.0 -0.082"/>
+    <origin rpy="0 0 0" xyz="-0.0 -0.0 -0.082"/>
     <geometry>
       <mesh filename="package://robotic_arm_description/meshes/link1_1.stl" scale="0.001 0.001 0.001"/>
@@ -46,10 +41,10 @@
 <link name="link2_1">
   <inertial>
-    <origin rpy="0 0 0" xyz="0.038703484335521884 -0.004887948983593355 0.03774231593240132"/>
+    <origin rpy="0 0 0" xyz="0.03900552900187564 -4.720497574409756e-08 0.03774797355252993"/>
     <mass value="8.491131635058604"/>
-    <inertia ixx="0.02803" ixy="3.5e-05" ixz="0.002251" iyy="0.028706" iyz="8.9e-05" izz="0.00947"/>
-  </inertial>
-  <visual>
-    <origin rpy="0 0 0" xyz="-0.024852 0.002717 -0.214"/>
+    <inertia ixx="0.028031" ixy="0.0" ixz="0.002228" iyy="0.028711" iyz="0.0" izz="0.009465"/>
+  </inertial>
+  <visual>
+    <origin rpy="0 0 0" xyz="-0.025 -0.0 -0.214"/>
     <geometry>
       <mesh filename="package://robotic_arm_description/meshes/link2_1.stl" scale="0.001 0.001 0.001"/>
@@ -58,5 +53,5 @@
   </visual>
   <collision>
-    <origin rpy="0 0 0" xyz="-0.024852 0.002717 -0.214"/>
+    <origin rpy="0 0 0" xyz="-0.025 -0.0 -0.214"/>
     <geometry>
       <mesh filename="package://robotic_arm_description/meshes/link2_1.stl" scale="0.001 0.001 0.001"/>
@@ -66,10 +61,10 @@
 <link name="link3_1">
   <inertial>
-    <origin rpy="0 0 0" xyz="0.012247659764739578 -0.0027447456236525426 0.09281098998429382"/>
+    <origin rpy="0 0 0" xyz="0.012475562747510771 1.9427211413704553e-08 0.09282105705277077"/>
     <mass value="8.19717066814797"/>
-    <inertia ixx="0.027202" ixy="5.4e-05" ixz="-0.001678" iyy="0.027457" iyz="0.000482" izz="0.008687"/>
-  </inertial>
-  <visual>
-    <origin rpy="0 0 0" xyz="-0.049456 0.007705 -0.34598"/>
+    <inertia ixx="0.027193" ixy="0.0" ixz="-0.001721" iyy="0.027471" iyz="0.0" izz="0.008682"/>
+  </inertial>
+  <visual>
+    <origin rpy="0 0 0" xyz="-0.05 -0.0 -0.346"/>
     <geometry>
       <mesh filename="package://robotic_arm_description/meshes/link3_1.stl" scale="0.001 0.001 0.001"/>
@@ -78,5 +73,5 @@
   </visual>
   <collision>
-    <origin rpy="0 0 0" xyz="-0.049456 0.007705 -0.34598"/>
+    <origin rpy="0 0 0" xyz="-0.05 -0.0 -0.346"/>
     <geometry>
       <mesh filename="package://robotic_arm_description/meshes/link3_1.stl" scale="0.001 0.001 0.001"/>
@@ -86,10 +81,10 @@
 <link name="link4_1">
   <inertial>
-    <origin rpy="0 0 0" xyz="-0.037264258405936466 0.004135664282855892 0.03916213989085432"/>
+    <origin rpy="0 0 0" xyz="-0.0374755647664739 1.4871117923491877e-08 0.03917892822918834"/>
     <mass value="8.197173492795319"/>
-    <inertia ixx="0.027191" ixy="-5e-06" ixz="-0.001739" iyy="0.027468" iyz="-0.000172" izz="0.008687"/>
-  </inertial>
-  <visual>
-    <origin rpy="0 0 0" xyz="-0.024313 0.007677 -0.477953"/>
+    <inertia ixx="0.027193" ixy="-0.0" ixz="-0.001721" iyy="0.027471" iyz="-0.0" izz="0.008682"/>
+  </inertial>
+  <visual>
+    <origin rpy="0 0 0" xyz="-0.025 -0.0 -0.478"/>
     <geometry>
       <mesh filename="package://robotic_arm_description/meshes/link4_1.stl" scale="0.001 0.001 0.001"/>
@@ -98,5 +93,5 @@
   </visual>
   <collision>
-    <origin rpy="0 0 0" xyz="-0.024313 0.007677 -0.477953"/>
+    <origin rpy="0 0 0" xyz="-0.025 -0.0 -0.478"/>
     <geometry>
       <mesh filename="package://robotic_arm_description/meshes/link4_1.stl" scale="0.001 0.001 0.001"/>
@@ -106,10 +101,10 @@
 <link name="link5_1">
   <inertial>
-    <origin rpy="0 0 0" xyz="-0.00039926406308956176 -0.012958499242889332 0.03618497852505709"/>
+    <origin rpy="0 0 0" xyz="5.829486113497266e-07 -0.013599717850522941 0.035950542831699184"/>
     <mass value="2.7272453464013666"/>
-    <inertia ixx="0.005718" ixy="-1.4e-05" ixz="4.7e-05" iyy="0.00527" iyz="0.001494" izz="0.003338"/>
-  </inertial>
-  <visual>
-    <origin rpy="0 0 0" xyz="0.000405 0.003056 -0.609925"/>
+    <inertia ixx="0.005718" ixy="0.0" ixz="-0.0" iyy="0.005217" iyz="0.001527" izz="0.003392"/>
+  </inertial>
+  <visual>
+    <origin rpy="0 0 0" xyz="0.0 -0.0 -0.61"/>
     <geometry>
       <mesh filename="package://robotic_arm_description/meshes/link5_1.stl" scale="0.001 0.001 0.001"/>
@@ -118,5 +113,5 @@
   </visual>
   <collision>
-    <origin rpy="0 0 0" xyz="0.000405 0.003056 -0.609925"/>
+    <origin rpy="0 0 0" xyz="0.0 -0.0 -0.61"/>
     <geometry>
       <mesh filename="package://robotic_arm_description/meshes/link5_1.stl" scale="0.001 0.001 0.001"/>
@@ -126,10 +121,10 @@
 <link name="link6_1">
   <inertial>
-    <origin rpy="0 0 0" xyz="0.0014434778410388274 0.043979261659800276 0.004989648922825052"/>
+    <origin rpy="0 0 0" xyz="1.2404412177094015e-07 0.043907868057215506 0.00576385697550974"/>
     <mass value="3.0329082890678123"/>
-    <inertia ixx="0.003349" ixy="-2.6e-05" ixz="-9e-06" iyy="0.002545" iyz="-0.000289" izz="0.002535"/>
-  </inertial>
-  <visual>
-    <origin rpy="0 0 0" xyz="0.001388 0.035799 -0.737522"/>
+    <inertia ixx="0.00335" ixy="0.0" ixz="-0.0" iyy="0.002555" iyz="-0.000289" izz="0.002524"/>
+  </inertial>
+  <visual>
+    <origin rpy="0 0 0" xyz="0.0 0.035 -0.737"/>
     <geometry>
       <mesh filename="package://robotic_arm_description/meshes/link6_1.stl" scale="0.001 0.001 0.001"/>
@@ -138,5 +133,5 @@
   </visual>
   <collision>
-    <origin rpy="0 0 0" xyz="0.001388 0.035799 -0.737522"/>
+    <origin rpy="0 0 0" xyz="0.0 0.035 -0.737"/>
     <geometry>
       <mesh filename="package://robotic_arm_description/meshes/link6_1.stl" scale="0.001 0.001 0.001"/>
@@ -144,81 +139,41 @@
   </collision>
 </link>
-<link name="gripper_base_1">
-  <inertial>
-    <origin rpy="0 0 0" xyz="0.005671804479930915 0.000408293874723218 0.015574536618465307"/>
-    <mass value="0.2541593681555956"/>
-    <inertia ixx="6e-05" ixy="-1e-06" ixz="-1.4e-05" iyy="7.8e-05" iyz="-1e-06" izz="5.2e-05"/>
-  </inertial>
-  <visual>
-    <origin rpy="0 0 0" xyz="-0.000563 -0.025218 -0.796456"/>
-    <geometry>
-      <mesh filename="package://robotic_arm_description/meshes/gripper_base_1.stl" scale="0.001 0.001 0.001"/>
-    </geometry>
-    <material name="silver"/>
-  </visual>
-  <collision>
-    <origin rpy="0 0 0" xyz="-0.000563 -0.025218 -0.796456"/>
-    <geometry>
-      <mesh filename="package://robotic_arm_description/meshes/gripper_base_1.stl" scale="0.001 0.001 0.001"/>
-    </geometry>
-  </collision>
-</link>
-<link name="jaw_base_1">
-  <inertial>
-    <origin rpy="0 0 0" xyz="-0.005493154029186715 -0.00012867837704213375 1.4021729310975672e-07"/>
-    <mass value="0.00550084263444652"/>
-    <inertia ixx="0.0" ixy="0.0" ixz="0.0" iyy="0.0" iyz="0.0" izz="0.0"/>
-  </inertial>
-  <visual>
-    <origin rpy="0 0 0" xyz="-0.00055 -0.025747 -0.826451"/>
-    <geometry>
-      <mesh filename="package://robotic_arm_description/meshes/jaw_base_1.stl" scale="0.001 0.001 0.001"/>
-    </geometry>
-    <material name="silver"/>
-  </visual>
-  <collision>
-    <origin rpy="0 0 0" xyz="-0.00055 -0.025747 -0.826451"/>
-    <geometry>
-      <mesh filename="package://robotic_arm_description/meshes/jaw_base_1.stl" scale="0.001 0.001 0.001"/>
-    </geometry>
-  </collision>
-</link>
-<link name="jaw_connector1_1">
-  <inertial>
-    <origin rpy="0 0 0" xyz="-0.0013520122931284916 0.014968776975824865 -0.00030912683646089345"/>
-    <mass value="0.0014253307496954507"/>
-    <inertia ixx="0.0" ixy="0.0" ixz="-0.0" iyy="0.0" iyz="0.0" izz="0.0"/>
-  </inertial>
-  <visual>
-    <origin rpy="0 0 0" xyz="0.006565 -0.030582 -0.826451"/>
-    <geometry>
-      <mesh filename="package://robotic_arm_description/meshes/jaw_connector1_1.stl" scale="0.001 0.001 0.001"/>
-    </geometry>
-    <material name="silver"/>
-  </visual>
-  <collision>
-    <origin rpy="0 0 0" xyz="0.006565 -0.030582 -0.826451"/>
-    <geometry>
-      <mesh filename="package://robotic_arm_description/meshes/jaw_connector1_1.stl" scale="0.001 0.001 0.001"/>
-    </geometry>
-  </collision>
-</link>
-<link name="jaw_connector2_1">
-  <inertial>
-    <origin rpy="0 0 0" xyz="-0.0006477588915065943 -0.015015832885347712 0.0003085573584135082"/>
-    <mass value="0.0014253307496953996"/>
-    <inertia ixx="0.0" ixy="0.0" ixz="-0.0" iyy="0.0" iyz="0.0" izz="0.0"/>
-  </inertial>
-  <visual>
-    <origin rpy="0 0 0" xyz="0.00633 -0.020584 -0.826451"/>
-    <geometry>
-      <mesh filename="package://robotic_arm_description/meshes/jaw_connector2_1.stl" scale="0.001 0.001 0.001"/>
-    </geometry>
-    <material name="silver"/>
-  </visual>
-  <collision>
-    <origin rpy="0 0 0" xyz="0.00633 -0.020584 -0.826451"/>
-    <geometry>
-      <mesh filename="package://robotic_arm_description/meshes/jaw_connector2_1.stl" scale="0.001 0.001 0.001"/>
+<link name="gripper_1">
+  <inertial>
+    <origin rpy="0 0 0" xyz="6.519052686577514e-09 -0.00043894585194131225 0.008806436122391847"/>
+    <mass value="0.14002124283631304"/>
+    <inertia ixx="2.9e-05" ixy="0.0" ixz="0.0" iyy="4.7e-05" iyz="1e-06" izz="4.2e-05"/>
+  </inertial>
+  <visual>
+    <origin rpy="0 0 0" xyz="-0.0 -0.025 -0.797"/>
+    <geometry>
+      <mesh filename="package://robotic_arm_description/meshes/gripper_1.stl" scale="0.001 0.001 0.001"/>
+    </geometry>
+    <material name="silver"/>
+  </visual>
+  <collision>
+    <origin rpy="0 0 0" xyz="-0.0 -0.025 -0.797"/>
+    <geometry>
+      <mesh filename="package://robotic_arm_description/meshes/gripper_1.stl" scale="0.001 0.001 0.001"/>
+    </geometry>
+  </collision>
+</link>
+<link name="jaw2_1">
+  <inertial>
+    <origin rpy="0 0 0" xyz="0.000131421896564822 0.0024996154528694157 0.015252945027369291"/>
+    <mass value="0.011516853958458544"/>
+    <inertia ixx="1e-06" ixy="0.0" ixz="-0.0" iyy="1e-06" iyz="-0.0" izz="0.0"/>
+  </inertial>
+  <visual>
+    <origin rpy="0 0 0" xyz="0.020495 -0.025 -0.843"/>
+    <geometry>
+      <mesh filename="package://robotic_arm_description/meshes/jaw2_1.stl" scale="0.001 0.001 0.001"/>
+    </geometry>
+    <material name="silver"/>
+  </visual>
+  <collision>
+    <origin rpy="0 0 0" xyz="0.020495 -0.025 -0.843"/>
+    <geometry>
+      <mesh filename="package://robotic_arm_description/meshes/jaw2_1.stl" scale="0.001 0.001 0.001"/>
     </geometry>
   </collision>
@@ -226,10 +181,10 @@
 <link name="jaw1_1">
   <inertial>
-    <origin rpy="0 0 0" xyz="0.0013067130636277464 -0.021646015407303536 0.04618696323663418"/>
-    <mass value="0.010774049361330109"/>
-    <inertia ixx="9e-06" ixy="-0.0" ixz="0.0" iyy="8e-06" iyz="2e-06" izz="1e-06"/>
-  </inertial>
-  <visual>
-    <origin rpy="0 0 0" xyz="0.007269 -0.060567 -0.825833"/>
+    <origin rpy="0 0 0" xyz="-0.0001314218965648116 0.0024996154528694157 0.015252945027369291"/>
+    <mass value="0.011516853958458544"/>
+    <inertia ixx="1e-06" ixy="0.0" ixz="0.0" iyy="1e-06" iyz="-0.0" izz="0.0"/>
+  </inertial>
+  <visual>
+    <origin rpy="0 0 0" xyz="-0.020495 -0.025 -0.843"/>
     <geometry>
       <mesh filename="package://robotic_arm_description/meshes/jaw1_1.stl" scale="0.001 0.001 0.001"/>
@@ -238,5 +193,5 @@
   </visual>
   <collision>
-    <origin rpy="0 0 0" xyz="0.007269 -0.060567 -0.825833"/>
+    <origin rpy="0 0 0" xyz="-0.020495 -0.025 -0.843"/>
     <geometry>
       <mesh filename="package://robotic_arm_description/meshes/jaw1_1.stl" scale="0.001 0.001 0.001"/>
@@ -244,65 +199,5 @@
   </collision>
 </link>
-<link name="jaw2_1">
-  <inertial>
-    <origin rpy="0 0 0" xyz="-0.0011789227138860239 0.023556620646007383 0.045204725144988855"/>
-    <mass value="0.011032989741009674"/>
-    <inertia ixx="9e-06" ixy="-0.0" ixz="-0.0" iyy="8e-06" iyz="-2e-06" izz="1e-06"/>
-  </inertial>
-  <visual>
-    <origin rpy="0 0 0" xyz="0.007625 0.009448 -0.827068"/>
-    <geometry>
-      <mesh filename="package://robotic_arm_description/meshes/jaw2_1.stl" scale="0.001 0.001 0.001"/>
-    </geometry>
-    <material name="silver"/>
-  </visual>
-  <collision>
-    <origin rpy="0 0 0" xyz="0.007625 0.009448 -0.827068"/>
-    <geometry>
-      <mesh filename="package://robotic_arm_description/meshes/jaw2_1.stl" scale="0.001 0.001 0.001"/>
-    </geometry>
-  </collision>
-</link>
-<link name="jaw2_1">
-  <inertial>
-    <origin rpy="0 0 0" xyz="-0.0023409227138860237 -0.012144379353992615 0.007827725144988862"/>
-    <mass value="0.011032989741009674"/>
-    <inertia ixx="9e-06" ixy="-0.0" ixz="-0.0" iyy="8e-06" iyz="-2e-06" izz="1e-06"/>
-  </inertial>
-  <visual>
-    <origin rpy="0 0 0" xyz="0.006463 -0.026253 -0.864445"/>
-    <geometry>
-      <mesh filename="package://robotic_arm_description/meshes/jaw2_1.stl" scale="0.001 0.001 0.001"/>
-    </geometry>
-    <material name="silver"/>
-  </visual>
-  <collision>
-    <origin rpy="0 0 0" xyz="0.006463 -0.026253 -0.864445"/>
-    <geometry>
-      <mesh filename="package://robotic_arm_description/meshes/jaw2_1.stl" scale="0.001 0.001 0.001"/>
-    </geometry>
-  </collision>
-</link>
-<link name="jaw1_1">
-  <inertial>
-    <origin rpy="0 0 0" xyz="-0.0014982869363722538 0.012620984592696467 0.007574963236634202"/>
-    <mass value="0.010774049361330109"/>
-    <inertia ixx="9e-06" ixy="-0.0" ixz="0.0" iyy="8e-06" iyz="2e-06" izz="1e-06"/>
-  </inertial>
-  <visual>
-    <origin rpy="0 0 0" xyz="0.004464 -0.0263 -0.864445"/>
-    <geometry>
-      <mesh filename="package://robotic_arm_description/meshes/jaw1_1.stl" scale="0.001 0.001 0.001"/>
-    </geometry>
-    <material name="silver"/>
-  </visual>
-  <collision>
-    <origin rpy="0 0 0" xyz="0.004464 -0.0263 -0.864445"/>
-    <geometry>
-      <mesh filename="package://robotic_arm_description/meshes/jaw1_1.stl" scale="0.001 0.001 0.001"/>
-    </geometry>
-  </collision>
-</link>
-<joint name="Rev20" type="continuous">
+<joint name="Rev11" type="continuous">
   <origin rpy="0 0 0" xyz="0.0 0.0 0.082"/>
   <parent link="base_link"/>
@@ -310,81 +205,56 @@
   <axis xyz="0.0 0.0 0.01"/>
 </joint>
-<joint name="Rev21" type="continuous">
-  <origin rpy="0 0 0" xyz="0.024852 -0.002717 0.132"/>
+<joint name="Rev12" type="revolute">
+  <origin rpy="0 0 0" xyz="0.025 0.0 0.132"/>
   <parent link="link1_1"/>
   <child link="link2_1"/>
-  <axis xyz="0.009941 -0.001087 -0.0"/>
-</joint>
-<joint name="Rev22" type="continuous">
-  <origin rpy="0 0 0" xyz="0.024604 -0.004988 0.13198"/>
+  <axis xyz="0.01 0.0 0.0"/>
+  <limit effort="100" lower="-1.570796" upper="1.570796" velocity="100"/>
+</joint>
+<joint name="Rev13" type="continuous">
+  <origin rpy="0 0 0" xyz="0.025 0.0 0.132"/>
   <parent link="link2_1"/>
   <child link="link3_1"/>
-  <axis xyz="-1.9e-05 -0.000172 0.009999"/>
-</joint>
-<joint name="Rev23" type="continuous">
-  <origin rpy="0 0 0" xyz="-0.025143 2.8e-05 0.131973"/>
+  <axis xyz="0.0 0.0 0.01"/>
+</joint>
+<joint name="Rev14" type="revolute">
+  <origin rpy="0 0 0" xyz="-0.025 0.0 0.132"/>
   <parent link="link3_1"/>
   <child link="link4_1"/>
-  <axis xyz="-0.009958 0.00092 -3e-06"/>
-</joint>
-<joint name="Rev24" type="continuous">
-  <origin rpy="0 0 0" xyz="-0.024718 0.004621 0.131972"/>
+  <axis xyz="-0.01 0.0 0.0"/>
+  <limit effort="100" lower="-1.570796" upper="1.570796" velocity="100"/>
+</joint>
+<joint name="Rev15" type="continuous">
+  <origin rpy="0 0 0" xyz="-0.025 0.0 0.132"/>
   <parent link="link4_1"/>
   <child link="link5_1"/>
-  <axis xyz="1.3e-05 0.000176 0.009998"/>
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
Commit message: Added smaple photos and videos.

File: src/robotic_arm_description/urdf/robotic_arm.xacro (robot description, xacro)
@@ -5,4 +5,9 @@
 <xacro:include filename="$(find robotic_arm_description)/urdf/robotic_arm.gazebo" />
 <link name="base_link">
+<inertial>
+    <origin rpy="0 0 0" xyz="-7.044926902746826e-09 -4.737750495934672e-09 0.038474409050025755"/>
+    <mass value="5.749401825671835"/>
+    <inertia ixx="0.007412" ixy="-0.0" ixz="-0.0" iyy="0.007412" iyz="-0.0" izz="0.008288"/>
+  </inertial>
   <visual>
     <origin rpy="0 0 0" xyz="0 0 0"/>

Commit message: roscontrollers added.

File: src/robotic_arm_description/urdf/robotic_arm.xacro (robot description, xacro)
@@ -204,4 +204,10 @@
   </collision>
 </link>
+  <!-- Used for fixing robot to Gazebo 'base_link' -->
+  <link name="world"/>
+<joint name="fixed" type="fixed">
+  <parent link="world"/>
+  <child link="base_link"/>
+</joint>
 <joint name="Rev11" type="continuous">
   <origin rpy="0 0 0" xyz="0.0 0.0 0.082"/>
